File: fuccs-shitty-addon.kicad/fuccs-shitty-addon.sch (KiCad schematic (older format))
At the start: 8 parts, among them J1 Shitty Addon + ISP, U1 ATtiny85-20SU

Commit message: Components placed
Parts:
- U1: value ATtiny85-20SU -> ATtiny85-20SUR
Changed lines of the file:
@@
 P 5700 3650
 F 0 "U1" H 5170 3696 50  0000 R CNN
-F 1 "ATtiny85-20SU" H 5170 3605 50  0000 R CNN
+F 1 "ATtiny85-20SUR" H 5170 3605 50  0000 R CNN
 F 2 "Housings_SOIC:SOIJ-8_5.3x5.3mm_Pitch1.27mm" H 5700 3650 50  0001 C CIN
 F 3 "http://ww1.microchip.com/downloads/en/DeviceDoc/atmel-2586-avr-8-bit-microcontroller-attiny25-attiny45-attiny85_datasheet.pdf" H 5700 3650 50  0001 C CNN
@@
 	8650 3050 8650 3400
 Wire Wire Line
-	8750 3400 8750 2950
+	8750 3400 8750 3050
 Text Label 8750 3400 1    50   ~ 0
 SDA_MOSI
 Wire Wire Line
-	8550 3400 8550 2950
+	8550 3400 8550 3200
 Wire Wire Line
-	8750 3900 8750 4350
+	8750 3900 8750 4250
 Text Label 8750 4250 1    50   ~ 0
 SCL_SCK
 Wire Wire Line
-	8550 3900 8550 4350
+	8550 3900 8550 4250
 Text Label 8550 4250 1    50   ~ 0
 ~RESET~

Commit message: Routing complete
Parts:
- J1: footprint Pin_Headers:Pin_Header_Straight_2x03_Pitch2.54mm_SMD -> fuccs-shitty-addon-footprints:Pin_Header_Straight_2x03_Pitch2.54mm_SMD_no-silk
Changed lines of the file:
@@
 F 0 "J1" H 8700 3917 50  0000 C CNN
 F 1 "Shitty Addon + ISP" H 8700 3826 50  0000 C CNN
-F 2 "Pin_Headers:Pin_Header_Straight_2x03_Pitch2.54mm_SMD" H 8650 3600 50  0001 C CNN
+F 2 "fuccs-shitty-addon-footprints:Pin_Header_Straight_2x03_Pitch2.54mm_SMD_no-silk" H 8650 3600 50  0001 C CNN
 F 3 "~" H 8650 3600 50  0001 C CNN
 	1    8650 3600
